File: Hardware/NekoPurrTech_TiltingCtrl.kicad_pcb (KiCad board)
At the start: 2 copper layers, 35 parts, among them IC1 TB67H450FNG, IC2 TPS70933DRVR, IC3 TPS70933DRVR, J1 Power_IN, J2 FMU_PWM, J3 Motor, J4 Dbg_Port, J5 Klicky, U1 STM32F030F4Px

Commit message: Finished Project
Parts:
- C1, C4, C6, R8: moved to B.Cu
- moved IC1 109.9 mm to (21.5, 20.0), turned to 90 degrees
- moved R8 108.8 mm to (21.6, 17.4), turned to 0 degrees
- moved R9 107.8 mm to (17.4, 17.7), turned to -90 degrees
- moved C12 107.8 mm to (19.1, 29.2)
- moved C5 107.8 mm to (15.2, 30.9)
- moved C8 107.8 mm to (19.1, 32.2)
- moved D1 107.8 mm to (27.9, 25.7)
- moved IC3 107.8 mm to (21.4, 29.2)
- moved J1 107.8 mm to (27.9, 30.2)
- moved J2 107.8 mm to (27.9, 22.6)
- moved J4 107.8 mm to (27.9, 35.4)
- moved C10 107.8 mm to (23.8, 29.2)
- moved C7 107.8 mm to (23.8, 32.2)
- moved IC2 107.8 mm to (21.4, 32.2)
- moved J3 107.8 mm to (15.2, 14.8)
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Connections:
- IC1 pad 6: /Motor+ -> /Motor-
- IC1 pad 8: /Motor- -> /Motor+
- J4 pad 2: /Dbg_TX -> /SWDIO
- J4 pad 3: /Dbg_RX -> /SWCLK
- J4 pad 4: /SWDIO -> /Dbg_RX
- J4 pad 5: /SWCLK -> /Dbg_TX
- U1 pad 11: /IN2 -> unconnected-(U1-PA5-Pad11)
- U1 pad 12: /ENC_A -> /ENC_B
- U1 pad 13: /ENC_B -> /ENC_A
- U1 pad 18: /FMU_PWM -> /Motor_PWM
- U1 pad 7: unconnected-(U1-PA1-Pad7) -> /IN2
Routing:
- net +3.3V_MCU: track 0.00 -> 45.8 mm, vias 0 -> 4
- net /ENC_B: track 0.00 -> 30.5 mm, vias 0 -> 1
- net +3.3V_ENC: track 0.00 -> 30.2 mm, vias 0 -> 2
- net /ENC_A: track 0.00 -> 29.2 mm, vias 0 -> 1
- net VCC: track 0.00 -> 28.7 mm, vias 0 -> 1
- net /Klicky: track 0.00 -> 20.8 mm
- net /Motor_PWM: track 0.00 -> 14.0 mm
- net /IN1: track 0.00 -> 13.5 mm, vias 0 -> 2
- net /SWDIO: track 0.00 -> 11.9 mm
- net /FMU_PWM_OUT: track 0.00 -> 11.1 mm
- net /IN2: track 0.00 -> 10.7 mm, vias 0 -> 2
- net /SWCLK: track 0.00 -> 10.7 mm
- net /Motor_PWM_OUT: track 0.00 -> 8.50 mm
- net /Motor-: track 0.00 -> 7.89 mm
- net /LED: track 0.00 -> 7.82 mm
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- added copper zone on B.Cu, net GND
- added copper zone on F.Cu, net GND
- added copper zone on B.Cu, net Net-(IC1-RS)
Other:
- board outline added: 16.3 x 24.2 mm
