File: Hardware/NekoPurrTech_TiltingCtrl.kicad_sch (KiCad schematic)
At the start: 34 parts, among them IC1 TB67H450FNG, IC2 TPS70933DRVR, IC3 TPS70933DRVR, J1 Power_IN, J2 FMU_PWM, J3 Motor, J4 Dbg_Port, J5 Klicky, U1 STM32F030F4Px

Commit message: Finished Project
Connections:
- net Dbg_RX: now also J4.4 (Pin_4); no longer J4.3 (Pin_3)
- net Dbg_TX: now also J4.5 (Pin_5); no longer J4.2 (Pin_2)
- net ENC_A: now also U1.13 (PA7); no longer U1.12 (PA6)
- net ENC_B: now also U1.12 (PA6); no longer U1.13 (PA7)
- net FMU_PWM: no longer U1.18 (PA10)
- net IN2: now also U1.7 (PA1); no longer U1.11 (PA5)
- net Motor+: now also IC1.8 (OUT2); no longer IC1.6 (OUT1)
- net Motor-: now also IC1.6 (OUT1); no longer IC1.8 (OUT2)
- net Motor_PWM: now also U1.18 (PA10)
- net SWCLK: now also J4.3 (Pin_3); no longer J4.5 (Pin_5)
- net SWDIO: now also J4.2 (Pin_2); no longer J4.4 (Pin_4)
Changed lines of the file:
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@@
 	)
 	(no_connect
-		(at 49.53 41.91)
-	)
-	(no_connect
 		(at 142.24 29.21)
 	)
@@
 	)
 	(no_connect
+		(at 49.53 52.07)
+	)
+	(no_connect
 		(at 53.34 184.15)
 	)
@@
 	(wire
 		(pts
-			(xy 49.53 52.07) (xy 63.5 52.07)
-		)
-		(stroke
-			(width 0)
-			(type default)
-		)
-	)
-	(wire
-		(pts
 			(xy 74.93 82.55) (xy 74.93 83.82)
 		)
@@
 	(wire
 		(pts
+			(xy 49.53 41.91) (xy 63.5 41.91)
+		)
+		(stroke
+			(width 0)
+			(type default)
+		)
+	)
+	(wire
+		(pts
 			(xy 81.28 22.86) (xy 74.93 22.86)
 		)
@@
 		)
 	)
-	(label "Motor_PWM_OUT"
-		(at 91.44 121.92 180)
+	(label "Motor-"
+		(at 201.93 114.3 180)
 		(fields_autoplaced yes)
 		(effects
@@
 		)
 	)
-	(label "NRST"
-		(at 13.97 39.37 0)
+	(label "Motor_PWM_OUT"
+		(at 91.44 121.92 180)
 		(fields_autoplaced yes)
 		(effects
@@
 				(size 1.27 1.27)
 			)
-			(justify left bottom)
+			(justify right bottom)
 		)
 	)
-	(label "BOOT0"
-		(at 85.09 82.55 0)
+	(label "NRST"
+		(at 13.97 39.37 0)
 		(fields_autoplaced yes)
 		(effects
@@
 		)
 	)
-	(label "Dbg_RX"
-		(at 125.73 180.34 0)
+	(label "BOOT0"
+		(at 85.09 82.55 0)
 		(fields_autoplaced yes)
 		(effects
@@
 		)
 	)
-	(label "Motor-"
-		(at 201.93 109.22 180)
+	(label "ENC_B"
+		(at 63.5 54.61 180)
 		(fields_autoplaced yes)
 		(effects
@@
 		)
 	)
-	(label "SWDIO"
-		(at 125.73 182.88 0)
-		(fields_autoplaced yes)
-		(effects
-			(font
-				(size 1.27 1.27)
-			)
-			(justify left bottom)
-		)
-	)
-	(label "ENC_B"
-		(at 63.5 57.15 180)
+	(label "Motor_PWM"
+		(at 63.5 62.23 180)
 		(fields_autoplaced yes)
 		(effects
@@
 		)
 	)
-	(label "IN2"
-		(at 63.5 52.07 180)
+	(label "IN1"
+		(at 63.5 49.53 180)
 		(fields_autoplaced yes)
 		(effects
@@
 		)
 	)
-	(label "IN1"
-		(at 63.5 49.53 180)
+	(label "Dbg_TX"
+		(at 63.5 44.45 180)
 		(fields_autoplaced yes)
 		(effects
@@
 		)
 	)
-	(label "Dbg_TX"
-		(at 63.5 44.45 180)
+	(label "ENC_A"
+		(at 90.17 180.34 0)
+		(fields_autoplaced yes)
+		(effects
+			(font
+				(size 1.27 1.27)
+			)
+			(justify left bottom)
+		)
+	)
+	(label "FMU_PWM_OUT"
+		(at 91.44 142.24 180)
 		(fields_autoplaced yes)
 		(effects
@@
 		)
 	)
-	(label "FMU_PWM"
-		(at 63.5 62.23 180)
+	(label "IN2"
+		(at 63.5 41.91 180)
 		(fields_autoplaced yes)
 		(effects
@@
 		)
 	)
-	(label "SWCLK"
-		(at 125.73 185.42 0)
+	(label "FMU_PWM"
+		(at 50.8 142.24 0)
 		(fields_autoplaced yes)
 		(effects
@@
 		)
 	)
-	(label "ENC_A"
-		(at 90.17 180.34 0)
+	(label "FMU_PWM"
+		(at 64.77 181.61 180)
 		(fields_autoplaced yes)
 		(effects
@@
 				(size 1.27 1.27)
 			)
-			(justify left bottom)
+			(justify right bottom)
 		)
 	)
-	(label "Dbg_TX"
-		(at 125.73 177.8 0)
+	(label "Dbg_RX"
+		(at 125.73 182.88 0)
 		(fields_autoplaced yes)
 		(effects
@@
 		)
 	)
-	(label "FMU_PWM_OUT"
-		(at 91.44 142.24 180)
+	(label "Klicky"
+		(at 63.5 39.37 180)
 		(fields_autoplaced yes)
 		(effects
@@
 		)
 	)
-	(label "FMU_PWM"
-		(at 50.8 142.24 0)
+	(label "OSCH_IN"
+		(at 13.97 49.53 0)
 		(fields_autoplaced yes)
 		(effects
@@
 		)
 	)
-	(label "FMU_PWM"
-		(at 64.77 181.61 180)
+	(label "BOOT0"
+		(at 13.97 44.45 0)
 		(fields_autoplaced yes)
 		(effects
@@
 				(size 1.27 1.27)
 			)
-			(justify right bottom)
+			(justify left bottom)
 		)
 	)
-	(label "Klicky"
-		(at 63.5 39.37 180)
+	(label "Dbg_TX"
+		(at 125.73 185.42 0)
 		(fields_autoplaced yes)
 		(effects
@@
 				(size 1.27 1.27)
 			)
-			(justify right bottom)
+			(justify left bottom)
 		)
 	)
-	(label "OSCH_IN"
-		(at 13.97 49.53 0)
+	(label "ENC_A"
+		(at 63.5 57.15 180)
 		(fields_autoplaced yes)
 		(effects
@@
 				(size 1.27 1.27)
 			)
-			(justify left bottom)
+			(justify right bottom)
 		)
 	)
-	(label "BOOT0"
-		(at 13.97 44.45 0)
+	(label "SWDIO"
+		(at 125.73 177.8 0)
 		(fields_autoplaced yes)
 		(effects
@@
 		)
 	)
-	(label "ENC_A"
-		(at 63.5 54.61 180)
+	(label "Motor+"
+		(at 201.93 109.22 180)
 		(fields_autoplaced yes)
 		(effects
@@
 		)
 	)
-	(label "Motor+"
-		(at 201.93 114.3 180)
+	(label "SWCLK"
+		(at 125.73 180.34 0)
 		(fields_autoplaced yes)
 		(effects
@@
 				(size 1.27 1.27)
 			)
-			(justify right bottom)
+			(justify left bottom)
 		)
 	)
